Commit message: added the new kinect cameras configuration

File: bacchus_gazebo/urdf/sensors.xacro (robot description, xacro)
@@ -242,14 +242,14 @@
     </xacro:unless>
   </gazebo>
-  <!-- Kinect v2 -->
-  <xacro:property name="kinect2_parent" value="base_link" />
-  <xacro:property name="kinect2_name" value="kinect2" />
-  <xacro:property name="kinect2_cam_px" value="0.45" />
-  <xacro:property name="kinect2_cam_py" value="0.0" />
-  <xacro:property name="kinect2_cam_pz" value="0.5" />
-  <xacro:property name="kinect2_cam_or" value="0.0" />
-  <xacro:property name="kinect2_cam_op" value="${M_PI/2}" />
-  <xacro:property name="kinect2_cam_oy" value="-${M_PI/2}" />
-  <link name="$(arg tf_prefix)${kinect2_name}_link">
+  <!-- Kinect v2 num 1-->
+  <xacro:property name="kinect2_1_parent" value="base_link" />
+  <xacro:property name="kinect2_1_name" value="kinect2_1" />
+  <xacro:property name="kinect2_1_cam_px" value="0" />
+  <xacro:property name="kinect2_1_cam_py" value="-0.2" />
+  <xacro:property name="kinect2_1_cam_pz" value="1.2" />
+  <xacro:property name="kinect2_1_cam_or" value="-${M_PI/2}" />
+  <xacro:property name="kinect2_1_cam_op" value="0" />
+  <xacro:property name="kinect2_1_cam_oy" value="-${M_PI/2}" />
+  <link name="$(arg tf_prefix)${kinect2_1_name}_link">
     <visual>
       <geometry>
@@ -270,23 +270,23 @@
     </inertial>
   </link>
-  <joint name="$(arg robot_name)_${kinect2_name}_joint" type="fixed">
-    <parent link="$(arg tf_prefix)${kinect2_parent}"/>
-    <child link="$(arg tf_prefix)${kinect2_name}_link"/>
-    <origin xyz="${kinect2_cam_px} ${kinect2_cam_py} ${kinect2_cam_pz}" rpy="${kinect2_cam_or} ${kinect2_cam_op} ${kinect2_cam_oy}"/>
-  </joint>
-  <link name="$(arg tf_prefix)${kinect2_name}_rgb_optical_frame"/>
-  <joint name="$(arg robot_name)_${kinect2_name}_rgb_joint" type="fixed">
-    <parent link="$(arg tf_prefix)${kinect2_name}_link"/>
-    <child link="$(arg tf_prefix)${kinect2_name}_rgb_optical_frame"/>
+  <joint name="$(arg robot_name)_${kinect2_1_name}_joint" type="fixed">
+    <parent link="$(arg tf_prefix)${kinect2_1_parent}"/>
+    <child link="$(arg tf_prefix)${kinect2_1_name}_link"/>
+    <origin xyz="${kinect2_1_cam_px} ${kinect2_1_cam_py} ${kinect2_1_cam_pz}" rpy="${kinect2_1_cam_or} ${kinect2_1_cam_op} ${kinect2_1_cam_oy}"/>
+  </joint>
+  <link name="$(arg tf_prefix)${kinect2_1_name}_rgb_optical_frame"/>
+  <joint name="$(arg robot_name)_${kinect2_1_name}_rgb_joint" type="fixed">
+    <parent link="$(arg tf_prefix)${kinect2_1_name}_link"/>
+    <child link="$(arg tf_prefix)${kinect2_1_name}_rgb_optical_frame"/>
     <origin xyz="0 0.0125 0.016" rpy="-1.57 0 -1.57"/>
   </joint>
-  <link name="$(arg tf_prefix)${kinect2_name}_depth_optical_frame"/>
-  <joint name="$(arg robot_name)_${kinect2_name}_depth_joint" type="fixed">
-    <parent link="$(arg tf_prefix)${kinect2_name}_link"/>
-    <child link="$(arg tf_prefix)${kinect2_name}_depth_optical_frame"/>
+  <link name="$(arg tf_prefix)${kinect2_1_name}_depth_optical_frame"/>
+  <joint name="$(arg robot_name)_${kinect2_1_name}_depth_joint" type="fixed">
+    <parent link="$(arg tf_prefix)${kinect2_1_name}_link"/>
+    <child link="$(arg tf_prefix)${kinect2_1_name}_depth_optical_frame"/>
     <origin xyz="0 -0.0125 0.016" rpy="-1.57 0 -1.57"/>
   </joint>
-  <gazebo reference="$(arg tf_prefix)${kinect2_name}_link">
-    <sensor name="$(arg robot_name)_${kinect2_name}_sensor" type="depth">
+  <gazebo reference="$(arg tf_prefix)${kinect2_1_name}_link">
+    <sensor name="$(arg robot_name)_${kinect2_1_name}_sensor" type="depth">
       <always_on>true</always_on>
       <update_rate>30.0</update_rate>
@@ -311,6 +311,6 @@
         </noise>
       </camera>
-      <plugin name="$(arg robot_name)_${kinect2_name}_sensor_controller" filename="libgazebo_ros_openni_kinect.so">
-        <cameraName>${kinect2_name}_sensor</cameraName>
+      <plugin name="$(arg robot_name)_${kinect2_1_name}_sensor_controller" filename="libgazebo_ros_openni_kinect.so">
+        <cameraName>${kinect2_1_name}_sensor</cameraName>
         <alwaysOn>true</alwaysOn>
         <updateRate>30.0</updateRate>
@@ -320,5 +320,5 @@
         <cameraInfoTopicName>sd/camera_info</cameraInfoTopicName>
         <!--<depthImageCameraInfoTopicName>depth/camera_info</depthImageCameraInfoTopicName>-->
-        <frameName>${kinect2_name}_depth_optical_frame</frameName>
+        <frameName>${kinect2_1_name}_depth_optical_frame</frameName>
         <pointCloudCutoff>0.5</pointCloudCutoff>
         <pointCloudCutoffMax>8.0</pointCloudCutoffMax>
@@ -333,9 +333,9 @@
     </sensor>
   </gazebo>
-  <gazebo reference="$(arg tf_prefix)${kinect2_name}_link">
-    <sensor name="$(arg robot_name)_${kinect2_name}_camera" type="camera">
+  <gazebo reference="$(arg tf_prefix)${kinect2_1_name}_link">
+    <sensor name="$(arg robot_name)_${kinect2_1_name}_camera" type="camera">
       <always_on>true</always_on>
       <update_rate>30.0</update_rate>
-      <camera name="${kinect2_name}_camera">
+      <camera name="${kinect2_1_name}_camera">
         <horizontal_fov>${84.1*3.14/180.0}</horizontal_fov>
         <image>
@@ -357,11 +357,11 @@
         </noise>
       </camera>
-      <plugin name="$(arg robot_name)_${kinect2_name}_camera_controller" filename="libgazebo_ros_camera.so">
+      <plugin name="$(arg robot_name)_${kinect2_1_name}_camera_controller" filename="libgazebo_ros_camera.so">
         <alwaysOn>true</alwaysOn>
         <updateRate>30.0</updateRate>
-        <cameraName>${kinect2_name}_camera</cameraName>
+        <cameraName>${kinect2_1_name}_camera</cameraName>
         <imageTopicName>hd/image_color_rect</imageTopicName>
         <cameraInfoTopicName>hd/camera_info</cameraInfoTopicName>
-        <frameName>${kinect2_name}_rgb_optical_frame</frameName>
+        <frameName>${kinect2_1_name}_rgb_optical_frame</frameName>
         <baseline>0.1</baseline>
         <distortionK1>0.0</distortionK1>
@@ -374,3 +374,135 @@
     </sensor>
   </gazebo>
+   <!-- Kinect v2 num 2-->
+  <xacro:property name="kinect2_2_parent" value="base_link" />
+  <xacro:property name="kinect2_2_name" value="kinect2_2" />
+  <xacro:property name="kinect2_2_cam_px" value="0" />
+  <xacro:property name="kinect2_2_cam_py" value="0.2" />
+  <xacro:property name="kinect2_2_cam_pz" value="1.2" />
+  <xacro:property name="kinect2_2_cam_or" value="${M_PI/2}" />
+  <xacro:property name="kinect2_2_cam_op" value="0" />
+  <xacro:property name="kinect2_2_cam_oy" value="${M_PI/2}" />
+  <link name="$(arg tf_prefix)${kinect2_2_name}_link">
+    <visual>
+      <geometry>
+        <mesh filename="package://kinect2_description/meshes/sensors/kinect2.dae"/>
+      </geometry>
+      <origin xyz="0.02 0 0" rpy="0 0 3.141592"/>
+    </visual>
+    <collision>
+      <geometry>
+        <box size=".1 .25 .06"/>
+      </geometry>
+      <contact_coefficients mu="0" kp="1000.0" kd="1.0"/>
+    </collision>
+    <inertial>
+      <mass value="1e-5" />
+      <origin xyz="0 0 0" rpy="0 0 0"/>
+      <inertia ixx="1e-6" ixy="0" ixz="0" iyy="1e-6" iyz="0" izz="1e-6" />
+    </inertial>
+  </link>
+  <joint name="$(arg robot_name)_${kinect2_2_name}_joint" type="fixed">
+    <parent link="$(arg tf_prefix)${kinect2_2_parent}"/>
+    <child link="$(arg tf_prefix)${kinect2_2_name}_link"/>
+    <origin xyz="${kinect2_2_cam_px} ${kinect2_2_cam_py} ${kinect2_2_cam_pz}" rpy="${kinect2_2_cam_or} ${kinect2_2_cam_op} ${kinect2_2_cam_oy}"/>
+  </joint>
+  <link name="$(arg tf_prefix)${kinect2_2_name}_rgb_optical_frame"/>
+  <joint name="$(arg robot_name)_${kinect2_2_name}_rgb_joint" type="fixed">
+    <parent link="$(arg tf_prefix)${kinect2_2_name}_link"/>
+    <child link="$(arg tf_prefix)${kinect2_2_name}_rgb_optical_frame"/>
+    <origin xyz="0 0.0125 0.016" rpy="-1.57 0 -1.57"/>
+  </joint>
+  <link name="$(arg tf_prefix)${kinect2_2_name}_depth_optical_frame"/>
+  <joint name="$(arg robot_name)_${kinect2_2_name}_depth_joint" type="fixed">
+    <parent link="$(arg tf_prefix)${kinect2_2_name}_link"/>
+    <child link="$(arg tf_prefix)${kinect2_2_name}_depth_optical_frame"/>
+    <origin xyz="0 -0.0125 0.016" rpy="-1.57 0 -1.57"/>
+  </joint>
+  <gazebo reference="$(arg tf_prefix)${kinect2_2_name}_link">
+    <sensor name="$(arg robot_name)_${kinect2_2_name}_sensor" type="depth">
+      <always_on>true</always_on>
+      <update_rate>30.0</update_rate>
+      <camera>
+        <horizontal_fov>${70.0*3.14/180.0}</horizontal_fov>
+        <image>
+          <width>512</width>
+          <height>424</height>
+          <format>L8</format>
+        </image>
+        <clip>
+          <near>0.1</near>
+          <far>8.0</far>
+        </clip>
+        <noise>
+          <!-- Noise is sampled independently per pixel on each frame.
+          That pixel's noise value is added to each of its color
+          channels, which at that point lie in the range [0,1]. -->
+          <type>gaussian</type>
+          <mean>0.0</mean>
+          <stddev>0.001</stddev>
+        </noise>
+      </camera>
+      <plugin name="$(arg robot_name)_${kinect2_2_name}_sensor_controller" filename="libgazebo_ros_openni_kinect.so">
+        <cameraName>${kinect2_2_name}_sensor</cameraName>
+        <alwaysOn>true</alwaysOn>
+        <updateRate>30.0</updateRate>
+        <imageTopicName>sd/image_ir_rect</imageTopicName>
+        <depthImageTopicName>sd/image_depth_rect</depthImageTopicName>
+        <pointCloudTopicName>sd/points</pointCloudTopicName>
+        <cameraInfoTopicName>sd/camera_info</cameraInfoTopicName>
+        <!--<depthImageCameraInfoTopicName>depth/camera_info</depthImageCameraInfoTopicName>-->
+        <frameName>${kinect2_2_name}_depth_optical_frame</frameName>
+        <pointCloudCutoff>0.5</pointCloudCutoff>
+        <pointCloudCutoffMax>8.0</pointCloudCutoffMax>
+        <baseline>0.1</baseline>
+        <distortionK1>0.0</distortionK1>
+        <distortionK2>0.0</distortionK2>
+        <distortionK3>0.0</distortionK3>
+        <distortionT1>0.0</distortionT1>
+        <distortionT2>0.0</distortionT2>
+        <robotNamespace>$(arg tf_prefix)</robotNamespace>
+      </plugin>
+    </sensor>
+  </gazebo>
+  <gazebo reference="$(arg tf_prefix)${kinect2_2_name}_link">
+    <sensor name="$(arg robot_name)_${kinect2_2_name}_camera" type="camera">
+      <always_on>true</always_on>
+      <update_rate>30.0</update_rate>
+      <camera name="${kinect2_2_name}_camera">
+        <horizontal_fov>${84.1*3.14/180.0}</horizontal_fov>
+        <image>
+          <width>1920</width>
+          <height>1080</height>
+          <format>R8G8B8</format>
+        </image>
+        <clip>
+          <near>0.02</near>
+          <far>10.0</far>
+        </clip>
+        <noise>
+          <!-- Noise is sampled independently per pixel on each frame.
+          That pixel's noise value is added to each of its color
+          channels, which at that point lie in the range [0,1]. -->
+          <type>gaussian</type>
+          <mean>0.0</mean>
+          <stddev>0.007</stddev>
+        </noise>
+      </camera>
+      <plugin name="$(arg robot_name)_${kinect2_2_name}_camera_controller" filename="libgazebo_ros_camera.so">
+        <alwaysOn>true</alwaysOn>
+        <updateRate>30.0</updateRate>
+        <cameraName>${kinect2_2_name}_camera</cameraName>
+        <imageTopicName>hd/image_color_rect</imageTopicName>
+        <cameraInfoTopicName>hd/camera_info</cameraInfoTopicName>
+        <frameName>${kinect2_2_name}_rgb_optical_frame</frameName>
+        <baseline>0.1</baseline>
+        <distortionK1>0.0</distortionK1>
+        <distortionK2>0.0</distortionK2>
+        <distortionK3>0.0</distortionK3>
+        <distortionT1>0.0</distortionT1>
+        <distortionT2>0.0</distortionT2>
+        <robotNamespace>$(arg tf_prefix)</robotNamespace>
+      </plugin>
+    </sensor>
+  </gazebo>
 </robot>
