Commit message: Remove fake sprayer. Modify hokuyo laser scanner location to the top right corner. Add another laser scanner to the bottom left corner. Modify the orientation + location of the kinect sensors. Add kinect sensor at the front of the robot.

File: bacchus_gazebo/urdf/sensors.xacro (robot description, xacro)
@@ -1,10 +1,12 @@
 <?xml version="1.0"?>
 <robot xmlns:xacro="http://www.ros.org/wiki/xacro" name="sensor_frames">
-	<!-- Import all sensors from sensors sub-folder -->
-	<xacro:include filename="$(find bacchus_gazebo)/urdf/sensors/sensor_fake_sprayer.xacro" />
-	<xacro:include filename="$(find bacchus_gazebo)/urdf/sensors/sensor_hokuyo_laser.xacro" />
-	<xacro:include filename="$(find bacchus_gazebo)/urdf/sensors/sensor_velodyne_vlp16.xacro" />
-	<xacro:include filename="$(find bacchus_gazebo)/urdf/sensors/sensor_kinect_v2_num1.xacro" />
-	<xacro:include filename="$(find bacchus_gazebo)/urdf/sensors/sensor_kinect_v2_num2.xacro" />
-	<xacro:include filename="$(find bacchus_gazebo)/urdf/sensors/sensor_imu.xacro" />
+  <!-- Import all sensors from sensors sub-folder -->
+  <!--xacro:include filename="$(find bacchus_gazebo)/urdf/sensors/sensor_fake_sprayer.xacro" /-->
+  <xacro:include filename="$(find bacchus_gazebo)/urdf/sensors/sensor_hokuyo_laser_top_right.xacro" />
+  <xacro:include filename="$(find bacchus_gazebo)/urdf/sensors/sensor_hokuyo_laser_bottom_left.xacro" />
+  <xacro:include filename="$(find bacchus_gazebo)/urdf/sensors/sensor_velodyne_vlp16.xacro" />
+  <xacro:include filename="$(find bacchus_gazebo)/urdf/sensors/sensor_kinect_v2_front.xacro" />
+  <xacro:include filename="$(find bacchus_gazebo)/urdf/sensors/sensor_kinect_v2_left.xacro" />
+  <xacro:include filename="$(find bacchus_gazebo)/urdf/sensors/sensor_kinect_v2_right.xacro" />
+  <xacro:include filename="$(find bacchus_gazebo)/urdf/sensors/sensor_imu.xacro" />
 </robot>

File: bacchus_gazebo/urdf/sensors/sensor_hokuyo_laser_bottom_left.xacro (robot description, xacro)
@@ -3,6 +3,9 @@
   <xacro:arg name="robot_name" default=""/>
   <xacro:arg name="tf_prefix" default=""/>
+  <xacro:property name="xyz" value="-0.7025 0.60 0.66"/>
+  <xacro:property name="rpy" value="0 0 -3.141592"/>
+  <xacro:property name="sensor_name" value="hokuyo_bottom_left"/>
   <!-- Hokuyo Laser -->
-  <link name="$(arg tf_prefix)hokuyo">
+  <link name="$(arg tf_prefix)${sensor_name}">
     <collision>
       <origin xyz="0 0 0" rpy="0 0 0"/>
@@ -23,13 +26,13 @@
     </inertial>
   </link>
-  <joint name="$(arg robot_name)_base_link_hokuyo" type="fixed">
+  <joint name="$(arg robot_name)_base_link_${sensor_name}" type="fixed">
     <parent link="$(arg tf_prefix)base_link"/>
-    <child link="$(arg tf_prefix)hokuyo"/>
+    <child link="$(arg tf_prefix)${sensor_name}"/>
     <axis xyz="0 1 0" />
-    <origin xyz="0.7025 0.005 0.66" rpy="0 0 0"/>
+    <origin xyz="${xyz}" rpy="${rpy}"/>
   </joint>
   <!--hokuyo-->
-  <gazebo reference="$(arg tf_prefix)hokuyo">
-    <sensor name="$(arg robot_name)hokuyo_sensor" type="ray">
+  <gazebo reference="$(arg tf_prefix)${sensor_name}">
+    <sensor name="$(arg robot_name)${sensor_name}_sensor" type="ray">
       <pose>0 0 0 0 0 0</pose>
       <visualize>false</visualize>
@@ -41,5 +44,5 @@
             <samples>720</samples>
             <resolution>1</resolution>
-            <min_angle>-1.570796</min_angle>
+            <min_angle>-3.141592</min_angle>
             <max_angle>1.570796</max_angle>
           </horizontal>
@@ -60,7 +63,7 @@
         </noise>
       </ray>
-      <plugin name="$(arg robot_name)hokuyo_node" filename="libgazebo_ros_laser.so">
-        <topicName>scan</topicName>
-        <frameName>hokuyo</frameName>
+      <plugin name="$(arg robot_name)${sensor_name}_node" filename="libgazebo_ros_laser.so">
+        <topicName>${sensor_name}_scan</topicName>
+        <frameName>${sensor_name}</frameName>
       </plugin>
     </sensor>

File: bacchus_gazebo/urdf/sensors/sensor_kinect_v2_left.xacro (robot description, xacro)
@@ -3,14 +3,14 @@
   <xacro:arg name="robot_name" default=""/>
   <xacro:arg name="tf_prefix" default=""/>
-   <!-- Kinect v2 num 2-->
-  <xacro:property name="kinect2_2_parent" value="base_link" />
-  <xacro:property name="kinect2_2_name" value="kinect2_2" />
-  <xacro:property name="kinect2_2_cam_px" value="0" />
-  <xacro:property name="kinect2_2_cam_py" value="0.2" />
-  <xacro:property name="kinect2_2_cam_pz" value="1.2" />
-  <xacro:property name="kinect2_2_cam_or" value="${M_PI/2}" />
-  <xacro:property name="kinect2_2_cam_op" value="0" />
-  <xacro:property name="kinect2_2_cam_oy" value="${M_PI/2}" />
-  <link name="$(arg tf_prefix)${kinect2_2_name}_link">
+  <!-- Kinect v2 -->
+  <xacro:property name="kinect2_parent" value="base_link" />
+  <xacro:property name="kinect2_name"   value="kinect2_left" />
+  <xacro:property name="kinect2_cam_px" value="0.0 " />
+  <xacro:property name="kinect2_cam_py" value="0.34" />
+  <xacro:property name="kinect2_cam_pz" value="0.80" />
+  <xacro:property name="kinect2_cam_or" value="0" />
+  <xacro:property name="kinect2_cam_op" value="0" />
+  <xacro:property name="kinect2_cam_oy" value="${90*M_PI/180}" />
+  <link name="$(arg tf_prefix)${kinect2_name}_link">
     <visual>
       <geometry>
@@ -31,23 +31,23 @@
     </inertial>
   </link>
-  <joint name="$(arg robot_name)_${kinect2_2_name}_joint" type="fixed">
-    <parent link="$(arg tf_prefix)${kinect2_2_parent}"/>
-    <child link="$(arg tf_prefix)${kinect2_2_name}_link"/>
-    <origin xyz="${kinect2_2_cam_px} ${kinect2_2_cam_py} ${kinect2_2_cam_pz}" rpy="${kinect2_2_cam_or} ${kinect2_2_cam_op} ${kinect2_2_cam_oy}"/>
+  <joint name="$(arg robot_name)_${kinect2_name}_joint" type="fixed">
+    <parent link="$(arg tf_prefix)${kinect2_parent}"/>
+    <child link="$(arg tf_prefix)${kinect2_name}_link"/>
+    <origin xyz="${kinect2_cam_px} ${kinect2_cam_py} ${kinect2_cam_pz}" rpy="${kinect2_cam_or} ${kinect2_cam_op} ${kinect2_cam_oy}"/>
   </joint>
-  <link name="$(arg tf_prefix)${kinect2_2_name}_rgb_optical_frame"/>
-  <joint name="$(arg robot_name)_${kinect2_2_name}_rgb_joint" type="fixed">
-    <parent link="$(arg tf_prefix)${kinect2_2_name}_link"/>
-    <child link="$(arg tf_prefix)${kinect2_2_name}_rgb_optical_frame"/>
+  <link name="$(arg tf_prefix)${kinect2_name}_rgb_optical_frame"/>
+  <joint name="$(arg robot_name)_${kinect2_name}_rgb_joint" type="fixed">
+    <parent link="$(arg tf_prefix)${kinect2_name}_link"/>
+    <child link="$(arg tf_prefix)${kinect2_name}_rgb_optical_frame"/>
     <origin xyz="0 0.0125 0.016" rpy="-1.57 0 -1.57"/>
   </joint>
-  <link name="$(arg tf_prefix)${kinect2_2_name}_depth_optical_frame"/>
-  <joint name="$(arg robot_name)_${kinect2_2_name}_depth_joint" type="fixed">
-    <parent link="$(arg tf_prefix)${kinect2_2_name}_link"/>
-    <child link="$(arg tf_prefix)${kinect2_2_name}_depth_optical_frame"/>
+  <link name="$(arg tf_prefix)${kinect2_name}_depth_optical_frame"/>
+  <joint name="$(arg robot_name)_${kinect2_name}_depth_joint" type="fixed">
+    <parent link="$(arg tf_prefix)${kinect2_name}_link"/>
+    <child link="$(arg tf_prefix)${kinect2_name}_depth_optical_frame"/>
     <origin xyz="0 -0.0125 0.016" rpy="-1.57 0 -1.57"/>
   </joint>
-  <gazebo reference="$(arg tf_prefix)${kinect2_2_name}_link">
-    <sensor name="$(arg robot_name)_${kinect2_2_name}_sensor" type="depth">
+  <gazebo reference="$(arg tf_prefix)${kinect2_name}_link">
+    <sensor name="$(arg robot_name)_${kinect2_name}_sensor" type="depth">
       <always_on>true</always_on>
       <update_rate>30.0</update_rate>
@@ -72,6 +72,6 @@
         </noise>
       </camera>
-      <plugin name="$(arg robot_name)_${kinect2_2_name}_sensor_controller" filename="libgazebo_ros_openni_kinect.so">
-        <cameraName>${kinect2_2_name}_sensor</cameraName>
+      <plugin name="$(arg robot_name)_${kinect2_name}_sensor_controller" filename="libgazebo_ros_openni_kinect.so">
+        <cameraName>${kinect2_name}_sensor</cameraName>
         <alwaysOn>true</alwaysOn>
         <updateRate>30.0</updateRate>
@@ -81,5 +81,5 @@
         <cameraInfoTopicName>sd/camera_info</cameraInfoTopicName>
         <!--<depthImageCameraInfoTopicName>depth/camera_info</depthImageCameraInfoTopicName>-->
-        <frameName>${kinect2_2_name}_depth_optical_frame</frameName>
+        <frameName>${kinect2_name}_depth_optical_frame</frameName>
         <pointCloudCutoff>0.5</pointCloudCutoff>
         <pointCloudCutoffMax>8.0</pointCloudCutoffMax>
@@ -94,9 +94,9 @@
     </sensor>
   </gazebo>
-  <gazebo reference="$(arg tf_prefix)${kinect2_2_name}_link">
-    <sensor name="$(arg robot_name)_${kinect2_2_name}_camera" type="camera">
+  <gazebo reference="$(arg tf_prefix)${kinect2_name}_link">
+    <sensor name="$(arg robot_name)_${kinect2_name}_camera" type="camera">
       <always_on>true</always_on>
       <update_rate>30.0</update_rate>
-      <camera name="${kinect2_2_name}_camera">
+      <camera name="${kinect2_name}_camera">
         <horizontal_fov>${84.1*3.14/180.0}</horizontal_fov>
         <image>
@@ -118,11 +118,11 @@
         </noise>
       </camera>
-      <plugin name="$(arg robot_name)_${kinect2_2_name}_camera_controller" filename="libgazebo_ros_camera.so">
+      <plugin name="$(arg robot_name)_${kinect2_name}_camera_controller" filename="libgazebo_ros_camera.so">
         <alwaysOn>true</alwaysOn>
         <updateRate>30.0</updateRate>
-        <cameraName>${kinect2_2_name}_camera</cameraName>
+        <cameraName>${kinect2_name}_camera</cameraName>
         <imageTopicName>hd/image_color_rect</imageTopicName>
         <cameraInfoTopicName>hd/camera_info</cameraInfoTopicName>
-        <frameName>${kinect2_2_name}_rgb_optical_frame</frameName>
+        <frameName>${kinect2_name}_rgb_optical_frame</frameName>
         <baseline>0.1</baseline>
         <distortionK1>0.0</distortionK1>

File: bacchus_gazebo/urdf/sensors/sensor_kinect_v2_right.xacro (robot description, xacro)
@@ -3,14 +3,14 @@
   <xacro:arg name="robot_name" default=""/>
   <xacro:arg name="tf_prefix" default=""/>
-  <!-- Kinect v2 num 1-->
-  <xacro:property name="kinect2_1_parent" value="base_link" />
-  <xacro:property name="kinect2_1_name" value="kinect2_1" />
-  <xacro:property name="kinect2_1_cam_px" value="0" />
-  <xacro:property name="kinect2_1_cam_py" value="-0.2" />
-  <xacro:property name="kinect2_1_cam_pz" value="1.2" />
-  <xacro:property name="kinect2_1_cam_or" value="-${M_PI/2}" />
-  <xacro:property name="kinect2_1_cam_op" value="0" />
-  <xacro:property name="kinect2_1_cam_oy" value="-${M_PI/2}" />
-  <link name="$(arg tf_prefix)${kinect2_1_name}_link">
+  <!-- Kinect v2 -->
+  <xacro:property name="kinect2_parent" value="base_link" />
+  <xacro:property name="kinect2_name"   value="kinect2_right" />
+  <xacro:property name="kinect2_cam_px" value="0.0 " />
+  <xacro:property name="kinect2_cam_py" value="-0.34" />
+  <xacro:property name="kinect2_cam_pz" value="0.80" />
+  <xacro:property name="kinect2_cam_or" value="0" />
+  <xacro:property name="kinect2_cam_op" value="0" />
+  <xacro:property name="kinect2_cam_oy" value="${270*M_PI/180}" />
+  <link name="$(arg tf_prefix)${kinect2_name}_link">
     <visual>
       <geometry>
@@ -31,23 +31,23 @@
     </inertial>
   </link>
-  <joint name="$(arg robot_name)_${kinect2_1_name}_joint" type="fixed">
-    <parent link="$(arg tf_prefix)${kinect2_1_parent}"/>
-    <child link="$(arg tf_prefix)${kinect2_1_name}_link"/>
-    <origin xyz="${kinect2_1_cam_px} ${kinect2_1_cam_py} ${kinect2_1_cam_pz}" rpy="${kinect2_1_cam_or} ${kinect2_1_cam_op} ${kinect2_1_cam_oy}"/>
+  <joint name="$(arg robot_name)_${kinect2_name}_joint" type="fixed">
+    <parent link="$(arg tf_prefix)${kinect2_parent}"/>
+    <child link="$(arg tf_prefix)${kinect2_name}_link"/>
+    <origin xyz="${kinect2_cam_px} ${kinect2_cam_py} ${kinect2_cam_pz}" rpy="${kinect2_cam_or} ${kinect2_cam_op} ${kinect2_cam_oy}"/>
   </joint>
-  <link name="$(arg tf_prefix)${kinect2_1_name}_rgb_optical_frame"/>
-  <joint name="$(arg robot_name)_${kinect2_1_name}_rgb_joint" type="fixed">
-    <parent link="$(arg tf_prefix)${kinect2_1_name}_link"/>
-    <child link="$(arg tf_prefix)${kinect2_1_name}_rgb_optical_frame"/>
+  <link name="$(arg tf_prefix)${kinect2_name}_rgb_optical_frame"/>
+  <joint name="$(arg robot_name)_${kinect2_name}_rgb_joint" type="fixed">
+    <parent link="$(arg tf_prefix)${kinect2_name}_link"/>
+    <child link="$(arg tf_prefix)${kinect2_name}_rgb_optical_frame"/>
     <origin xyz="0 0.0125 0.016" rpy="-1.57 0 -1.57"/>
   </joint>
-  <link name="$(arg tf_prefix)${kinect2_1_name}_depth_optical_frame"/>
-  <joint name="$(arg robot_name)_${kinect2_1_name}_depth_joint" type="fixed">
-    <parent link="$(arg tf_prefix)${kinect2_1_name}_link"/>
-    <child link="$(arg tf_prefix)${kinect2_1_name}_depth_optical_frame"/>
+  <link name="$(arg tf_prefix)${kinect2_name}_depth_optical_frame"/>
+  <joint name="$(arg robot_name)_${kinect2_name}_depth_joint" type="fixed">
+    <parent link="$(arg tf_prefix)${kinect2_name}_link"/>
+    <child link="$(arg tf_prefix)${kinect2_name}_depth_optical_frame"/>
     <origin xyz="0 -0.0125 0.016" rpy="-1.57 0 -1.57"/>
   </joint>
-  <gazebo reference="$(arg tf_prefix)${kinect2_1_name}_link">
-    <sensor name="$(arg robot_name)_${kinect2_1_name}_sensor" type="depth">
+  <gazebo reference="$(arg tf_prefix)${kinect2_name}_link">
+    <sensor name="$(arg robot_name)_${kinect2_name}_sensor" type="depth">
       <always_on>true</always_on>
       <update_rate>30.0</update_rate>
@@ -72,6 +72,6 @@
         </noise>
       </camera>
-      <plugin name="$(arg robot_name)_${kinect2_1_name}_sensor_controller" filename="libgazebo_ros_openni_kinect.so">
-        <cameraName>${kinect2_1_name}_sensor</cameraName>
+      <plugin name="$(arg robot_name)_${kinect2_name}_sensor_controller" filename="libgazebo_ros_openni_kinect.so">
+        <cameraName>${kinect2_name}_sensor</cameraName>
         <alwaysOn>true</alwaysOn>
         <updateRate>30.0</updateRate>
@@ -81,5 +81,5 @@
         <cameraInfoTopicName>sd/camera_info</cameraInfoTopicName>
         <!--<depthImageCameraInfoTopicName>depth/camera_info</depthImageCameraInfoTopicName>-->
-        <frameName>${kinect2_1_name}_depth_optical_frame</frameName>
+        <frameName>${kinect2_name}_depth_optical_frame</frameName>
         <pointCloudCutoff>0.5</pointCloudCutoff>
         <pointCloudCutoffMax>8.0</pointCloudCutoffMax>
@@ -94,9 +94,9 @@
     </sensor>
   </gazebo>
-  <gazebo reference="$(arg tf_prefix)${kinect2_1_name}_link">
-    <sensor name="$(arg robot_name)_${kinect2_1_name}_camera" type="camera">
+  <gazebo reference="$(arg tf_prefix)${kinect2_name}_link">
+    <sensor name="$(arg robot_name)_${kinect2_name}_camera" type="camera">
       <always_on>true</always_on>
       <update_rate>30.0</update_rate>
-      <camera name="${kinect2_1_name}_camera">
+      <camera name="${kinect2_name}_camera">
         <horizontal_fov>${84.1*3.14/180.0}</horizontal_fov>
         <image>
@@ -118,11 +118,11 @@
         </noise>
       </camera>
-      <plugin name="$(arg robot_name)_${kinect2_1_name}_camera_controller" filename="libgazebo_ros_camera.so">
+      <plugin name="$(arg robot_name)_${kinect2_name}_camera_controller" filename="libgazebo_ros_camera.so">
         <alwaysOn>true</alwaysOn>
         <updateRate>30.0</updateRate>
-        <cameraName>${kinect2_1_name}_camera</cameraName>
+        <cameraName>${kinect2_name}_camera</cameraName>
         <imageTopicName>hd/image_color_rect</imageTopicName>
         <cameraInfoTopicName>hd/camera_info</cameraInfoTopicName>
-        <frameName>${kinect2_1_name}_rgb_optical_frame</frameName>
+        <frameName>${kinect2_name}_rgb_optical_frame</frameName>
         <baseline>0.1</baseline>
         <distortionK1>0.0</distortionK1>
