Commit message: Parametrised hokuyo + 2 sensors suites
The test should now pass

File: bacchus_gazebo/urdf/bacchus_sensors.xacro (robot description, xacro)
@@ -12,10 +12,18 @@
           xyz="0 0 1.5"
           rpy="0 0 0"/>
-  <xacro:hokuyo sensor_name="hokuyo_bottom_left"
-          xyz="-0.7025 0.6 0.66"
-          rpy="0 0 0"/>
-  <xacro:hokuyo sensor_name="hokuyo_top_right"
-          xyz="0.7025 -0.6 0.66"
-          rpy="0 0 ${-M_PI}"/>
+  <xacro:hokuyo sensor_name="hokuyo_back"
+          xyz="0.172 -0.152 -0.034"
+          rpy="0 0 -0.79"
+          min_angle="-2.18"
+          max_angle="2.36"
+          hokuyo_parent="top3"
+          topic="back_scan"/>
+  <xacro:hokuyo sensor_name="hokuyo_front"
+          xyz="0.172 -0.152 -0.034"
+          rpy="0 0 -0.79"
+          min_angle="-2.18"
+          max_angle="2.36"
+          hokuyo_parent="top1"
+          topic="front_scan"/>
   <xacro:kinect kinect2_name="kinect2_front"
           kinect2_cam_px="0.5025"

File: bacchus_gazebo/urdf/sensors/sensor_hokuyo_laser.xacro (robot description, xacro)
@@ -4,6 +4,5 @@
   <xacro:arg name="tf_prefix" default="" />
   <xacro:property name="M_PI" value="3.1415926535897931" />
-  <xacro:property name="hokuyo_parent" value="base_link" />
-  <xacro:macro name="hokuyo" params="xyz rpy sensor_name">
+  <xacro:macro name="hokuyo" params="xyz rpy min_angle max_angle sensor_name hokuyo_parent topic">
     <!-- <xacro:property name="xyz" value="0.7025 -0.6 0.66" />
     <xacro:property name="rpy" value="0 0 0" />
@@ -29,5 +28,5 @@
     </inertial>
     </link>
-    <joint name="$(arg robot_name)_base_link_${sensor_name}" type="fixed">
+    <joint name="$(arg robot_name)_${hokuyo_parent}_${sensor_name}" type="fixed">
       <parent link="$(arg tf_prefix)${hokuyo_parent}" />
       <child link="$(arg tf_prefix)${sensor_name}" />
@@ -47,6 +46,6 @@
               <samples>720</samples>
               <resolution>1</resolution>
-              <min_angle>-2.39</min_angle>
-              <max_angle>2.39</max_angle>
+              <min_angle>${min_angle}</min_angle>
+              <max_angle>${max_angle}</max_angle>
             </horizontal>
           </scan>
@@ -67,5 +66,5 @@
         </ray>
         <plugin name="$(arg robot_name)${sensor_name}_node" filename="libgazebo_ros_laser.so">
-          <topicName>${sensor_name}_scan</topicName>
+          <topicName>${topic}</topicName>
           <frameName>${sensor_name}</frameName>
         </plugin>
