Commit message: Add gaussian noise to imu

File: bacchus_gazebo/urdf/sensors/sensor_imu.xacro (robot description, xacro)
@@ -27,5 +27,5 @@
     <child link="$(arg tf_prefix)imu_sensor_link"/>
     <axis xyz="0 1 0" />
-    <origin xyz="0 0 1.56" rpy="0 0 0"/>
+    <origin xyz="0 0 1.65" rpy="0 0 0"/>
   </joint>
   <gazebo reference="$(arg tf_prefix)imu_sensor_link">
@@ -33,5 +33,5 @@
 		<sensor name="$(arg robot_name)imu_sensor" type="imu">
 			<always_on>true</always_on>
-			<update_rate>500</update_rate>
+			<update_rate>1000</update_rate>
 			<visualize>true</visualize>
 			<topic>__default_topic__</topic>
@@ -39,5 +39,5 @@
 				<topicName>imu_raw</topicName>
 				<bodyName>imu_sensor_link</bodyName>
-				<updateRateHZ>10.0</updateRateHZ>
+				<updateRateHZ>500.0</updateRateHZ>
 				<gaussianNoise>0.0</gaussianNoise>
 				<xyzOffset>0 0 0</xyzOffset>
@@ -48,4 +48,58 @@
 			<pose>0 0 0 0 0 0</pose>
 			<material>Gazebo/Orange</material>
+        <imu_sensor>
+          <angular_velocity>
+            <x>
+              <noise type="gaussian">
+                <mean>0.0</mean>
+                <stddev>2e-4</stddev>
+                <bias_mean>0.0000075</bias_mean>
+                <bias_stddev>0.0000008</bias_stddev>
+              </noise>
+            </x>
+            <y>
+              <noise type="gaussian">
+                <mean>0.0</mean>
+                <stddev>2e-4</stddev>
+                <bias_mean>0.0000075</bias_mean>
+                <bias_stddev>0.0000008</bias_stddev>
+              </noise>
+            </y>
+            <z>
+              <noise type="gaussian">
+                <mean>0.0</mean>
+                <stddev>2e-4</stddev>
+                <bias_mean>0.0000075</bias_mean>
+                <bias_stddev>0.0000008</bias_stddev>
+              </noise>
+            </z>
+          </angular_velocity>
+          <linear_acceleration>
+            <x>
+              <noise type="gaussian">
+                <mean>0.0</mean>
+                <stddev>1.7e-2</stddev>
+                <bias_mean>0.1</bias_mean>
+                <bias_stddev>0.001</bias_stddev>
+              </noise>
+            </x>
+            <y>
+              <noise type="gaussian">
+                <mean>0.0</mean>
+                <stddev>1.7e-2</stddev>
+                <bias_mean>0.1</bias_mean>
+                <bias_stddev>0.001</bias_stddev>
+              </noise>
+            </y>
+            <z>
+              <noise type="gaussian">
+                <mean>0.0</mean>
+                <stddev>1.7e-2</stddev>
+                <bias_mean>0.1</bias_mean>
+                <bias_stddev>0.001</bias_stddev>
+              </noise>
+            </z>
+          </linear_acceleration>
+        </imu_sensor>
 		</sensor>
 	</gazebo>

Commit message: try to add plugin for hector imu plugin

File: bacchus_gazebo/urdf/sensors/sensor_imu.xacro (robot description, xacro)
@@ -48,6 +48,25 @@
           <initialOrientationAsReference>false</initialOrientationAsReference>
         </plugin>
-        <pose>0 0 0 0 0 0</pose>
-        <material>Gazebo/Orange</material>
+        <!--plugin name="$(arg robot_name)imu_sensor" filename="libhector_gazebo_ros_imu.so">
+          <serviceName>/imu/calibrate</serviceName>
+          <alwaysOn>true</alwaysOn>
+          <robotNamespace>/$(arg robot_name)</robotNamespace>
+          <updateRate>1000</updateRate>
+          <bodyName>${sensor_name}</bodyName>
+          <frameId>$(arg tf_prefix)${sensor_name}</frameId>
+          <topicName>imu_raw</topicName>
+          <rpyOffset>0 0 0</rpyOffset>
+          <xyzOffset>0 0 0</xyzOffset>
+          <gaussianNoise>0.00000001</gaussianNoise>
+          <accelDrift>0.00000001 0.00000001 0.00000001</accelDrift>
+          <accelDriftFrequency>0.00000001 0.00000001 0.00000001</accelDriftFrequency>
+          <accelGaussianNoise>0.00000001 0.00000001 0.00000001</accelGaussianNoise>
+          <rateDrift>0.0 0.0 0.0</rateDrift>
+          <rateDriftFrequency>0.0 0.0 0.0</rateDriftFrequency>
+          <rateGaussianNoise>0.0 0.0 0.0</rateGaussianNoise>
+          <headingDrift>0.0 0.0 0.0</headingDrift>
+          <headingDriftFrequency>0.0 0.0 0.0</headingDriftFrequency>
+          <headingGaussianNoise>0.0 0.0 0.0</headingGaussianNoise>
+        </plugin-->
         <!--imu_sensor>
           <angular_velocity>
@@ -106,4 +125,4 @@
       </sensor>
     </gazebo>
-    </xacro:macro>
+  </xacro:macro>
 </robot>
