Commit message: update kinect baseline

File: bacchus_gazebo/urdf/sensors/sensor_kinect_v2.xacro (robot description, xacro)
@@ -36,5 +36,5 @@
       <parent link="$(arg tf_prefix)${kinect2_name}_link" />
       <child link="$(arg tf_prefix)${kinect2_name}_rgb_optical_frame" />
-      <origin xyz="0 0.0125 0.016" rpy="-1.57 0 -1.57" />
+      <origin xyz="0 0.05 0.016" rpy="-1.57 0 -1.57" />
     </joint>
     <link name="$(arg tf_prefix)${kinect2_name}_depth_optical_frame" />
@@ -42,5 +42,5 @@
       <parent link="$(arg tf_prefix)${kinect2_name}_link" />
       <child link="$(arg tf_prefix)${kinect2_name}_depth_optical_frame" />
-      <origin xyz="0 -0.0125 0.016" rpy="-1.57 0 -1.57" />
+      <origin xyz="0 -0.05 0.016" rpy="-1.57 0 -1.57" />
     </joint>
     <gazebo reference="$(arg tf_prefix)${kinect2_name}_link">

Commit message: Modify kinect_v2 sensor file
* Rename the topics 
* Modify the RGB and Depth frame sizes to be the same size 640x480

File: bacchus_gazebo/urdf/sensors/sensor_kinect_v2.xacro (robot description, xacro)
@@ -36,5 +36,5 @@
       <parent link="$(arg tf_prefix)${kinect2_name}_link" />
       <child link="$(arg tf_prefix)${kinect2_name}_rgb_optical_frame" />
-      <origin xyz="0 0.0125 0.016" rpy="-1.57 0 -1.57" />
+      <origin xyz="0 0.05 0.016" rpy="-1.57 0 -1.57" />
     </joint>
     <link name="$(arg tf_prefix)${kinect2_name}_depth_optical_frame" />
@@ -42,5 +42,5 @@
       <parent link="$(arg tf_prefix)${kinect2_name}_link" />
       <child link="$(arg tf_prefix)${kinect2_name}_depth_optical_frame" />
-      <origin xyz="0 -0.0125 0.016" rpy="-1.57 0 -1.57" />
+      <origin xyz="0 -0.05 0.016" rpy="-1.57 0 -1.57" />
     </joint>
     <gazebo reference="$(arg tf_prefix)${kinect2_name}_link">
@@ -51,6 +51,6 @@
           <horizontal_fov>${70.0*3.14/180.0}</horizontal_fov>
           <image>
-            <width>512</width>
-            <height>424</height>
+            <width>640</width>
+            <height>480</height>
             <format>L8</format>
           </image>
@@ -72,10 +72,10 @@
           <alwaysOn>true</alwaysOn>
           <updateRate>30.0</updateRate>
-          <imageTopicName>sd/image_ir_rect</imageTopicName>
-          <depthImageTopicName>sd/image_depth_rect</depthImageTopicName>
-          <pointCloudTopicName>sd/points</pointCloudTopicName>
-          <cameraInfoTopicName>sd/camera_info</cameraInfoTopicName>
+          <imageTopicName>ir/image_ir_rect</imageTopicName>
+          <depthImageTopicName>ir/depth/image_raw</depthImageTopicName>
+          <pointCloudTopicName>ir/points</pointCloudTopicName>
+          <cameraInfoTopicName>ir/camera_info</cameraInfoTopicName>
           <!--<depthImageCameraInfoTopicName>depth/camera_info</depthImageCameraInfoTopicName>-->
-          <frameName>/${kinect2_name}_depth_optical_frame</frameName>
+          <frameName>${kinect2_name}_depth_optical_frame</frameName>
           <pointCloudCutoff>0.5</pointCloudCutoff>
           <pointCloudCutoffMax>8.0</pointCloudCutoffMax>
@@ -97,6 +97,6 @@
           <horizontal_fov>${84.1*3.14/180.0}</horizontal_fov>
           <image>
-            <width>1920</width>
-            <height>1080</height>
+            <width>640</width>
+            <height>480</height>
             <format>R8G8B8</format>
           </image>
@@ -118,7 +118,7 @@
           <updateRate>30.0</updateRate>
           <cameraName>${kinect2_name}_camera</cameraName>
-          <imageTopicName>hd/image_color_rect</imageTopicName>
-          <cameraInfoTopicName>hd/camera_info</cameraInfoTopicName>
-          <frameName>/${kinect2_name}_rgb_optical_frame</frameName>
+          <imageTopicName>rgb/image_raw</imageTopicName>
+          <cameraInfoTopicName>rgb/camera_info</cameraInfoTopicName>
+          <frameName>${kinect2_name}_rgb_optical_frame</frameName>
           <baseline>0.1</baseline>
           <distortionK1>0.0</distortionK1>

Commit message: added image, rtab_rgb_slam and corrected kinect2 model

File: bacchus_gazebo/urdf/sensors/sensor_kinect_v2.xacro (robot description, xacro)
@@ -42,5 +42,5 @@
       <parent link="$(arg tf_prefix)${kinect2_name}_link" />
       <child link="$(arg tf_prefix)${kinect2_name}_depth_optical_frame" />
-      <origin xyz="0 -0.05 0.016" rpy="-1.57 0 -1.57" />
+      <origin xyz="0 0.05 0.016" rpy="-1.57 0 -1.57" />
     </joint>
     <gazebo reference="$(arg tf_prefix)${kinect2_name}_link">
@@ -95,5 +95,5 @@
         <update_rate>30.0</update_rate>
         <camera name="${kinect2_name}_camera">
-          <horizontal_fov>${84.1*3.14/180.0}</horizontal_fov>
+          <horizontal_fov>${70.1*3.14/180.0}</horizontal_fov>
           <image>
             <width>640</width>
