Commit message: increase velodyne resolutoin to 1800 and enable GPU

File: bacchus_gazebo/urdf/sensors/sensor_velodyne_vlp16.xacro (robot description, xacro)
@@ -8,5 +8,5 @@
   <xacro:property name="velodyne_hz" value="10" />
   <xacro:property name="velodyne_lasers" value="16" />
-  <xacro:property name="velodyne_samples" value="440" />
+  <xacro:property name="velodyne_samples" value="1800" />
   <xacro:property name="velodyne_collision_range" value="0.3" />
   <xacro:property name="velodyne_min_range" value="0.9" />
@@ -15,5 +15,5 @@
   <xacro:property name="velodyne_min_angle" value="-${M_PI}" />
   <xacro:property name="velodyne_max_angle" value="${M_PI}" />
-  <xacro:property name="velodyne_gpu" value="false" />
+  <xacro:property name="velodyne_gpu" value="true" />
   <xacro:macro name="VLP-16" params="xyz rpy velodyne_name" >
     <link name="$(arg tf_prefix)${velodyne_name}_link">

Commit message: increase velodyne resolution + enable gpu flag

File: bacchus_gazebo/urdf/sensors/sensor_velodyne_vlp16.xacro (robot description, xacro)
@@ -6,14 +6,14 @@
   <xacro:property name="velodyne_parent" value="base_link" />
   <xacro:property name="velodyne_topic" value="velodyne_points" />
-  <xacro:property name="velodyne_hz" value="10" />
+  <xacro:property name="velodyne_hz" value="15" />
   <xacro:property name="velodyne_lasers" value="16" />
-  <xacro:property name="velodyne_samples" value="440" />
+  <xacro:property name="velodyne_samples" value="3600" />
   <xacro:property name="velodyne_collision_range" value="0.3" />
   <xacro:property name="velodyne_min_range" value="0.9" />
-  <xacro:property name="velodyne_max_range" value="130.0" />
+  <xacro:property name="velodyne_max_range" value="100.0" />
   <xacro:property name="velodyne_noise" value="0.008" />
   <xacro:property name="velodyne_min_angle" value="-${M_PI}" />
   <xacro:property name="velodyne_max_angle" value="${M_PI}" />
-  <xacro:property name="velodyne_gpu" value="false" />
+  <xacro:property name="velodyne_gpu" value="true" />
   <xacro:macro name="VLP-16" params="xyz rpy velodyne_name" >
     <link name="$(arg tf_prefix)${velodyne_name}_link">

Commit message: fix tf for velodyne

File: bacchus_gazebo/urdf/sensors/sensor_velodyne_vlp16.xacro (robot description, xacro)
@@ -6,7 +6,7 @@
   <xacro:property name="velodyne_parent" value="base_link" />
   <xacro:property name="velodyne_topic" value="velodyne_points" />
-  <xacro:property name="velodyne_hz" value="15" />
+  <xacro:property name="velodyne_hz" value="10" />
   <xacro:property name="velodyne_lasers" value="16" />
-  <xacro:property name="velodyne_samples" value="3600" />
+  <xacro:property name="velodyne_samples" value="1800" />
   <xacro:property name="velodyne_collision_range" value="0.3" />
   <xacro:property name="velodyne_min_range" value="0.9" />
@@ -99,5 +99,5 @@
           <plugin name="gazebo_ros_laser_controller" filename="libgazebo_ros_velodyne_gpu_laser.so">
             <topicName>${velodyne_topic}</topicName>
-            <frameName>$(arg tf_prefix)${velodyne_name}</frameName>
+            <frameName>/${velodyne_name}</frameName>
             <min_range>${velodyne_min_range}</min_range>
             <max_range>${velodyne_max_range}</max_range>
@@ -139,5 +139,5 @@
           <plugin name="gazebo_ros_laser_controller" filename="libgazebo_ros_velodyne_laser.so">
             <topicName>${velodyne_topic}</topicName>
-            <frameName>$(arg tf_prefix)${velodyne_name}</frameName>
+            <frameName>/${velodyne_name}</frameName>
             <min_range>${velodyne_min_range}</min_range>
             <max_range>${velodyne_max_range}</max_range>
