Commit message: Rename liosam base_link

File: LIO-SAM/launch/include/config/robot.urdf.xacro (robot description, xacro)
@@ -3,7 +3,7 @@
   <xacro:property name="PI" value="3.1415926535897931" />
   <link name="chassis_link"></link>
-  <link name="base_link"></link>
-  <joint name="base_link_joint" type="fixed">
-    <parent link="base_link"/>
+  <link name="base_link_lio"></link>
+  <joint name="base_link_lio_joint" type="fixed">
+    <parent link="base_link_lio"/>
     <child link="chassis_link" />
     <origin xyz="0 0 0" rpy="0 0 0" />
